Commit message: fix for AIRO-353: Correct the gripper mesh file names in Niryo URDF

File: tutorials/pick_and_place/PickAndPlaceProject/Assets/URDF/niryo_one/niryo_one.urdf (robot description, URDF)
Before this commit: robot niryo_one, 15 links, 13 joints
Links:
- link left_gripper: geometry collision mesh filename=package://niryo_one_urdf/Gripper1/G1_ClampLeft.STL scale=.001 .001 .001; visual mesh filename=package://niryo_one_urdf/Gripper1/G1_ClampLeft.STL scale=.001 .001 .001
- link right_gripper: geometry collision mesh filename=package://niryo_one_urdf/Gripper1/G1_ClampRight.STL scale=.001 .001 .001; visual mesh filename=package://niryo_one_urdf/Gripper1/G1_ClampRight.STL scale=.001 .001 .001
Joints:
- joint control_rod_left: origin xyz=0 0 0 rpy=0 3.141 0 -> xyz=0 0 0 rpy=0 0 0
- joint control_rod_right: origin xyz=0 0 0 rpy=0 0 0 -> xyz=0 0 0 rpy=0 3.141 0
- joint gripper_joint_left: limit lower=-2.57436 upper=2.57436 effort=1 velocity=1.0 -> lower=-0.0257436 upper=0.0257436 effort=1 velocity=1.0; origin xyz=0 0 0 rpy=0 3.141 0 -> xyz=0 0 0 rpy=0 0 0
- joint gripper_joint_right: limit lower=-2.57436 upper=2.57436 effort=1 velocity=1.0 -> lower=-0.0257436 upper=0.0257436 effort=1 velocity=1.0; origin xyz=0 0 0 rpy=0 0 0 -> xyz=0 0 0 rpy=0 3.141 0
